Commit message: Initial commit. so_arm_ros2_bridge provides a bridge for interacting with a physical SO-ARM10x LeRobot arm.

File: src/lerobot_description/urdf/so101_base.xacro (robot description, xacro)
@@ -4,4 +4,12 @@
   https://github.com/TheRobotStudio/SO-ARM100
   and has been modified accordingly.
+  Joint naming updated to match LeRobot motor conventions:
+    shoulder_pan_joint   (was "1")  base → shoulder
+    shoulder_lift_joint  (was "2")  shoulder → upper_arm
+    elbow_flex_joint     (was "3")  upper_arm → lower_arm
+    wrist_flex_joint     (was "4")  lower_arm → wrist
+    wrist_roll_joint     (was "5")  wrist → gripper
+    gripper_joint        (was "6")  gripper → gripper_finger
+  Link "jaw" renamed to "gripper_finger" to match LeRobot naming.
 -->
 <robot xmlns:xacro="http://www.ros.org/wiki/xacro">
@@ -275,5 +283,5 @@
 		</collision>
 	</link>
-	<!-- Link gripper -->
+	<!-- Link gripper (wrist_roll assembly, carries motor 5) -->
 	<link name="gripper">
 		<inertial>
@@ -316,6 +324,6 @@
 		</collision>
 	</link>
-	<!-- Link jaw -->
-	<link name="jaw">
+	<!-- Link gripper_finger (mobile jaw, driven by motor 6) -->
+	<link name="gripper_finger">
 		<inertial>
 			<origin xyz="-0.00157495 -0.0300244 0.0192755" rpy="0 0 0" />
@@ -339,15 +347,15 @@
 		</collision>
 	</link>
-	<!-- Joint from gripper to jaw -->
-	<joint name="6" type="revolute">
+	<!-- Joint from gripper to gripper_finger (motor 6 — LeRobot: gripper) -->
+	<joint name="gripper_joint" type="revolute">
 		<origin xyz="0.0202 0.0188 -0.0234" rpy="1.5708 -5.14108e-17 -1.38655e-14" />
 		<parent link="gripper" />
-		<child link="jaw" />
+		<child link="gripper_finger" />
 		<axis xyz="0 0 1" />
 		<limit effort="10" velocity="10" lower="-0.174533" upper="1.74533" />
 	</joint>
-	<transmission name="6_trans">
-		<type>transmission_interface/SimpleTransmission</type>
-		<joint name="6">
+	<transmission name="gripper_joint_trans">
+		<type>transmission_interface/SimpleTransmission</type>
+		<joint name="gripper_joint">
 			<hardwareInterface>hardware_interface/PositionJointInterface</hardwareInterface>
 		</joint>
@@ -357,6 +365,6 @@
 		</actuator>
 	</transmission>
-	<!-- Joint from wrist to gripper -->
-	<joint name="5" type="revolute">
+	<!-- Joint from wrist to gripper (motor 5 — LeRobot: wrist_roll) -->
+	<joint name="wrist_roll_joint" type="revolute">
 		<origin xyz="0 -0.0611 0.0181" rpy="1.5708 -9.38083e-08 3.14159" />
 		<parent link="wrist" />
@@ -365,7 +373,7 @@
 		<limit effort="10" velocity="10" lower="-2.79253" upper="2.79253" />
 	</joint>
-	<transmission name="5_trans">
-		<type>transmission_interface/SimpleTransmission</type>
-		<joint name="5">
+	<transmission name="wrist_roll_joint_trans">
+		<type>transmission_interface/SimpleTransmission</type>
+		<joint name="wrist_roll_joint">
 			<hardwareInterface>hardware_interface/PositionJointInterface</hardwareInterface>
 		</joint>
@@ -375,6 +383,6 @@
 		</actuator>
 	</transmission>
-	<!-- Joint from lower_arm to wrist -->
-	<joint name="4" type="revolute">
+	<!-- Joint from lower_arm to wrist (motor 4 — LeRobot: wrist_flex) -->
+	<joint name="wrist_flex_joint" type="revolute">
 		<origin xyz="-0.1349 0.0052 1.65232e-16" rpy="3.2474e-15 2.86219e-15 -1.5708" />
 		<parent link="lower_arm" />
@@ -383,7 +391,7 @@
 		<limit effort="10" velocity="10" lower="-1.65806" upper="1.65806" />
 	</joint>
-	<transmission name="4_trans">
-		<type>transmission_interface/SimpleTransmission</type>
-		<joint name="4">
+	<transmission name="wrist_flex_joint_trans">
+		<type>transmission_interface/SimpleTransmission</type>
+		<joint name="wrist_flex_joint">
 			<hardwareInterface>hardware_interface/PositionJointInterface</hardwareInterface>
 		</joint>
@@ -393,6 +401,6 @@
 		</actuator>
 	</transmission>
-	<!-- Joint from upper_arm to lower_arm -->
-	<joint name="3" type="revolute">
+	<!-- Joint from upper_arm to lower_arm (motor 3 — LeRobot: elbow_flex) -->
+	<joint name="elbow_flex_joint" type="revolute">
 		<origin xyz="-0.11257 -0.028 2.46331e-16" rpy="-1.22818e-15 5.75928e-16 1.5708" />
 		<parent link="upper_arm" />
@@ -401,7 +409,7 @@
 		<limit effort="10" velocity="10" lower="-1.74533" upper="1.5708" />
 	</joint>
-	<transmission name="3_trans">
-		<type>transmission_interface/SimpleTransmission</type>
-		<joint name="3">
+	<transmission name="elbow_flex_joint_trans">
+		<type>transmission_interface/SimpleTransmission</type>
+		<joint name="elbow_flex_joint">
 			<hardwareInterface>hardware_interface/PositionJointInterface</hardwareInterface>
 		</joint>
@@ -411,6 +419,6 @@
 		</actuator>
 	</transmission>
-	<!-- Joint from shoulder to upper_arm -->
-	<joint name="2" type="revolute">
+	<!-- Joint from shoulder to upper_arm (motor 2 — LeRobot: shoulder_lift) -->
+	<joint name="shoulder_lift_joint" type="revolute">
 		<origin xyz="-0.0303992 -0.0182778 -0.0542" rpy="-1.5708 -1.5708 0" />
 		<parent link="shoulder" />
@@ -419,7 +427,7 @@
 		<limit effort="10" velocity="10" lower="-1.74533" upper="1.74533" />
 	</joint>
-	<transmission name="2_trans">
-		<type>transmission_interface/SimpleTransmission</type>
-		<joint name="2">
+	<transmission name="shoulder_lift_joint_trans">
+		<type>transmission_interface/SimpleTransmission</type>
+		<joint name="shoulder_lift_joint">
 			<hardwareInterface>hardware_interface/PositionJointInterface</hardwareInterface>
 		</joint>
@@ -429,6 +437,6 @@
 		</actuator>
 	</transmission>
-	<!-- Joint from base to shoulder -->
-	<joint name="1" type="revolute">
+	<!-- Joint from base to shoulder (motor 1 — LeRobot: shoulder_pan) -->
+	<joint name="shoulder_pan_joint" type="revolute">
 		<origin xyz="0.0207909 -0.0230745 0.0948817" rpy="-3.14159 6.03684e-16 1.5708" />
 		<parent link="base" />
@@ -437,7 +445,7 @@
 		<limit effort="10" velocity="10" lower="-1.91986" upper="1.91986" />
 	</joint>
-	<transmission name="1_trans">
-		<type>transmission_interface/SimpleTransmission</type>
-		<joint name="1">
+	<transmission name="shoulder_pan_joint_trans">
+		<type>transmission_interface/SimpleTransmission</type>
+		<joint name="shoulder_pan_joint">
 			<hardwareInterface>hardware_interface/PositionJointInterface</hardwareInterface>
 		</joint>
